File: hardware/prism/prism.sch (EAGLE design)
At the start: 174 parts, among them IC1 XMEGA128-A1, IC2 74LVC4245APW, IC3 LM2731XMF, IC4 74LVC4245APW, IC5 LM25011MY, IC6 NCV78M05BDTRKG, IC7 NRF24L01+, IC8 MAX3232CSE, T1 MMBT2222LT1G, T2 NTGS4111PT1G, T3 MMBT2222LT1G, T4 MMBT2222LT1G, T5 NTGS4111PT1G, T6 MMBT2222LT1G, T7 MMBT2222LT1G, T8 NTGS4111PT1G

Commit message: bord routed, ready to review
Connections:
- removed net LED_EAST: IC1.PH1(!CAS!/!RE!)
- removed net LED_NORTH: IC1.PH7(CLK/!CS3!/A19)
- removed net LED_WEST: IC1.PA0(ADCA0/AREFA)
- removed net N$32: IC1.PJ3(D3/A3/A11), R40.1
- removed net N$36: IC1.PJ1(D1/A1/A9), R32.2
- new net LOW_BAT_LED_3V3: IC1.PE1(OC0B/XCK0/SCL), R40.1
- new net SYNC1_LED_3V3: IC1.PE0(OC0A/SDA), R32.2
- net BEACON_ID_0_3V3: now also IC1.PH2(!RAS!/ALE1); no longer IC1.PB0(ADCB0/AREFB)
- net BEACON_ID_1_3V3: now also IC1.PH3(!DOM!/ALE2); no longer IC1.PB1(ADCB1)
- net BEACON_ID_2_3V3: now also IC1.PH4(BA0/!CS0!/A16); no longer IC1.PB2(ADCB2/DAC0)
- net INT0_0_3V3: now also IC1.PE4(OC1A/!SS!), IC4.IO_VL4; no longer IC4.IO_VL5
- net INT0_1_3V3: now also IC1.PE5(OC1B/XCK1/MOSI), IC4.IO_VL5; no longer IC4.IO_VL4
- net INT1_0_3V3: now also IC1.PE6(RSC1/MISO/TOSC2), IC4.IO_VL6; no longer IC4.IO_VL3
- net INT1_1_3V3: now also IC1.PE7(TSD1/SCK/CLKO/EVO/TOSC1), IC4.IO_VL7; no longer IC4.IO_VL2
- net IR_SENSOR_0_OUTPUT_3V3: now also IC1.PD5(OC1B/XCK1/MOSI); no longer IC1.PC2(OC0C/RXD0)
- net IR_SENSOR_1_OUTPUT_3V3: now also IC1.PC0(OC0A/SDA); no longer IC1.PE2(OC0C/RXD0)
- net LED_INDEX_0_3V3: now also IC1.PB1(ADCB1); no longer IC1.PK6(A6/A14/A22)
- net LED_INDEX_1_3V3: now also IC1.PH0(!WE!); no longer IC1.PK7(A7/A15/A23)
- net LK0_3V3: now also IC1.PB2(ADCB2/DAC0); no longer IC1.PK0(A0/A8/A16)
- net LK1_3V3: now also IC1.PB3(ADCB3/DAC1); no longer IC1.PK1(A1/A9/A17)
- net LK2_3V3: now also IC1.PB4(ADCB4/TMS); no longer IC1.PK2(A2/A10/A18)
- net LK3_3V3: now also IC1.PB5(ADCB5/TDI); no longer IC1.PK3(A3/A11/A19)
- net LK4_3V3: now also IC1.PB6(ADCB6/TCK); no longer IC1.PK4(A4/A12/A20)
- net LK5_3V3: now also IC1.PB7(ADCB7/AC0-OUT/TDO); no longer IC1.PK5(A5/A13/A22)
- net MIRROR_INDEX_0_3V3: now also IC1.PD4(OC1A/!SS!); no longer IC1.PC3(OC0D/TXD0)
- net MIRROR_INDEX_1_3V3: now also IC1.PC3(OC0D/TXD0), IC1.PC4(OC1A/!SS!); no longer IC1.PE3(OC0D/TXD0)
- net N$10: now also IC1.PH5(BA1/!CS1!/A17); no longer IC1.PJ6(A10/D6/A6/A14)
- net N$12: now also IC1.PH7(CLK/!CS3!/A19); no longer IC1.PJ7(A11/D7/A7/A15)
- net N$28: now also IC1.PA6(ADCA6); no longer IC1.PJ0(D0/A0/A8)
- net N$31: now also IC1.PH1(!CAS!/!RE!); no longer IC1.PJ2(D2/A2/A10)
- net N$47: now also IC4.IO_VCC7; no longer IC4.IO_VCC2
- net N$53: now also IC4.IO_VCC6; no longer IC4.IO_VCC3
- net N$54: now also IC4.IO_VCC4; no longer IC4.IO_VCC5
- net N$55: now also IC4.IO_VCC5; no longer IC4.IO_VCC4
- net N$9: now also IC1.PH6(CKE/!CS2!/A18); no longer IC1.PJ5(A9/D5/A5/A13)
- net NRF_CSN_3V3: now also IC1.PA7/(ADCA7/AC0-OUT); no longer IC1.PE0(OC0A/SDA)
- net NRF_MOSI_3V3: now also IC1.PC5(OC1B/MOSI/XCK1); no longer IC1.PD5(OC1B/XCK1/MOSI)
- net ON/OFF_SENSOR_0_3V3: now also IC1.PD7(TXD1/SCK/CLKO/EVO); no longer IC1.PD2(OC0C/RXD0)
- net ON/OFF_SENSOR_1_3V3: now also IC1.PC2(OC0C/RXD0); no longer IC1.PD3(OC0D/TXD0)
- net RX_0_3V3: now also IC1.PF2(OC0C/RXD0), R30.2; no longer IC1.PF6(RXD1/MISO), R37.1
- net RX_1_3V3: now also IC1.PF6(RXD1/MISO), R37.1; no longer IC1.PF2(OC0C/RXD0), R30.2
- net SYNC_IN_0_3V3: now also IC1.PD2(OC0C/RXD0); no longer IC1.PC4(OC1A/!SS!)
- net SYNC_IN_1_3V3: now also IC1.PD6(RXD1/MISO); no longer IC1.PC5(OC1B/MOSI/XCK1)
- net SYNC_OUT_0_3V3: now also IC1.PF5(OC1B/XCK1/MOSI), IC4.IO_VL0; no longer IC1.PC6(MISO/RXD1), IC4.IO_VL6
- net SYNC_OUT_0_5V: now also IC4.IO_VCC0; no longer IC4.IO_VCC6
- net SYNC_OUT_1_3V3: now also IC1.PF4(OC1A/!SS!), IC4.IO_VL1; no longer IC1.PC7(SCK/TXD1/CLKO/EVO), IC4.IO_VL7
- net SYNC_OUT_1_5V: now also IC4.IO_VCC1; no longer IC4.IO_VCC7
- net TX_0_3V3: now also IC1.PF3(OC0D/TXD0), R33.2; no longer IC1.PF7(TXD1/SCK), R39.1
- net TX_1_3V3: now also IC1.PF7(TXD1/SCK), R39.1; no longer IC1.PF3(OC0D/TXD0), R33.2
- net XBEE_CTS_3V3/NRF_IRQ_3V3: now also IC1.PC1(OC0B/XCK0/SCL); no longer IC1.PH2(!RAS!/ALE1)
- net XBEE_RTS_3V3/NRF_CE_3V3: now also IC1.PB0(ADCB0/AREFB); no longer IC1.PH3(!DOM!/ALE2)
- net XBEE_RX_3V3/NRF_MISO_3V3: now also IC1.PC6(MISO/RXD1); no longer IC1.PD6(RXD1/MISO)
- net XBEE_TX_3V3/NRF_SCK_3V3: now also IC1.PC7(SCK/TXD1/CLKO/EVO); no longer IC1.PD7(TXD1/SCK/CLKO/EVO)
Other:
- note added: "use internal pullup of atxmega to read beacon id"
- note removed: "use internal pullup of atxmega"
- moved on the sheet: COM, ERROR, LOW_BATT, R1, R2, R25, R28, R30, R31, R32, R33, R35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

Commit message: ir index polarization resistor value changed after Damien review of prism_idx_suport board
Parts:
- R17: value 270-F -> 100-E; device robotter_resistor:270-F -> robotter_resistor:100-E
- R24: value 4K7-F -> 270-E; device robotter_resistor:4K7-F -> robotter_resistor:270-E
Other:
- note added: "3,3V 1A"
Changed lines of the file:
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@@
 <part name="+3V6" library="supply1" deviceset="+3V3" device=""/>
 <part name="+3V9" library="supply1" deviceset="+3V3" device=""/>
-<part name="R24" library="robotter_resistor" deviceset="4K7" device="-F"/>
-<part name="R17" library="robotter_resistor" deviceset="270" device="-F"/>
+<part name="R24" library="robotter_resistor" deviceset="270" device="-E"/>
+<part name="R17" library="robotter_resistor" deviceset="100" device="-E"/>
 <part name="GND5" library="supply1" deviceset="GND" device=""/>
 <part name="C18" library="robotter_capacitor" deviceset="100NF" device="-F" value="100nF 50V"/>
@@
 <text x="292.1" y="96.52" size="1.778" layer="91">SW_BATT is a switch used to drive the mos that cut power</text>
 <text x="279.4" y="-167.64" size="1.778" layer="91">led used to show idx activity</text>
+<text x="492.76" y="162.56" size="1.778" layer="91">3,3V 1A</text>
 </plain>
 <instances>
