File: hardware/prism/prism.sch (EAGLE design)
At the start: 174 parts, among them IC1 XMEGA128-A1, IC2 74LVC4245APW, IC3 LM2731XMF, IC4 74LVC4245APW, IC5 LM25011MY, IC6 NCV78M05BDTRKG, IC7 NRF24L01+, IC8 MAX3232CSE, T1 MMBT2222LT1G, T2 NTGS4111PT1G, T3 MMBT2222LT1G, T4 MMBT2222LT1G, T5 NTGS4111PT1G, T6 MMBT2222LT1G, T7 MMBT2222LT1G, T8 NTGS4111PT1G

Commit message: board update after Damien review
Connections:
- net GND: now also IC5.THERMAL_GND
- net SYNC_IN_0_3V3: now also IC1.PE2(OC0C/RXD0); no longer IC1.PD2(OC0C/RXD0)
Changed lines of the file:
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@@
 <instance part="SYNC1" gate="G$1" x="220.98" y="269.24" rot="R90"/>
 <instance part="R32" gate="G$1" x="208.28" y="269.24" rot="R180"/>
-<instance part="IC5" gate="G$1" x="444.5" y="142.24"/>
+<instance part="IC5" gate="G$1" x="444.5" y="144.78"/>
 <instance part="R6" gate="G$1" x="55.88" y="-96.52" smashed="yes">
 <attribute name="NAME" x="53.34" y="-93.98" size="1.778" layer="95"/>
@@
 <instance part="R72" gate="G$1" x="487.68" y="127" rot="R270"/>
 <instance part="R71" gate="G$1" x="487.68" y="142.24" rot="R270"/>
-<instance part="GND24" gate="1" x="444.5" y="116.84"/>
+<instance part="GND24" gate="1" x="447.04" y="116.84"/>
 <instance part="GND25" gate="1" x="462.28" y="134.62"/>
 <instance part="IC6" gate="G$1" x="444.5" y="99.06"/>
@@
 <wire x1="408.94" y1="119.38" x2="426.72" y2="119.38" width="0.1524" layer="91"/>
 <wire x1="426.72" y1="119.38" x2="444.5" y2="119.38" width="0.1524" layer="91"/>
-<wire x1="444.5" y1="119.38" x2="444.5" y2="127" width="0.1524" layer="91"/>
+<wire x1="444.5" y1="119.38" x2="447.04" y2="119.38" width="0.1524" layer="91"/>
+<wire x1="447.04" y1="119.38" x2="447.04" y2="127" width="0.1524" layer="91"/>
 <pinref part="C33" gate="G$1" pin="2"/>
 <wire x1="426.72" y1="124.46" x2="426.72" y2="119.38" width="0.1524" layer="91"/>
-<wire x1="444.5" y1="119.38" x2="487.68" y2="119.38" width="0.1524" layer="91"/>
+<wire x1="447.04" y1="119.38" x2="487.68" y2="119.38" width="0.1524" layer="91"/>
 <pinref part="R72" gate="G$1" pin="2"/>
 <wire x1="487.68" y1="119.38" x2="487.68" y2="121.92" width="0.1524" layer="91"/>
 <junction x="426.72" y="119.38"/>
-<junction x="444.5" y="119.38"/>
+<junction x="447.04" y="119.38"/>
 <pinref part="C29" gate="G$1" pin="2"/>
 <wire x1="408.94" y1="144.78" x2="408.94" y2="119.38" width="0.1524" layer="91"/>
@@
 <junction x="487.68" y="119.38"/>
 <junction x="408.94" y="119.38"/>
+<pinref part="IC5" gate="G$1" pin="THERMAL_GND"/>
+<wire x1="444.5" y1="127" x2="444.5" y2="119.38" width="0.1524" layer="91"/>
+<junction x="444.5" y="119.38"/>
 </segment>
 <segment>
 <pinref part="IC5" gate="G$1" pin="CSG"/>
-<wire x1="454.66" y1="139.7" x2="454.66" y2="137.16" width="0.1524" layer="91"/>
 <pinref part="R64" gate="G$1" pin="1"/>
-<wire x1="454.66" y1="137.16" x2="462.28" y2="137.16" width="0.1524" layer="91"/>
+<wire x1="457.2" y1="139.7" x2="457.2" y2="137.16" width="0.1524" layer="91"/>
+<wire x1="457.2" y1="137.16" x2="462.28" y2="137.16" width="0.1524" layer="91"/>
 <pinref part="GND25" gate="1" pin="GND"/>
 <junction x="462.28" y="137.16"/>
@@
 <pinref part="IC5" gate="G$1" pin="SW"/>
 <pinref part="D7" gate="G$1" pin="C"/>
-<wire x1="462.28" y1="152.4" x2="454.66" y2="152.4" width="0.1524" layer="91"/>
+<wire x1="462.28" y1="152.4" x2="457.2" y2="152.4" width="0.1524" layer="91"/>
 <pinref part="C36" gate="G$1" pin="2"/>
 <junction x="462.28" y="152.4"/>
@@
 <pinref part="IC5" gate="G$1" pin="CS"/>
 <pinref part="D7" gate="G$1" pin="A"/>
-<wire x1="462.28" y1="147.32" x2="454.66" y2="147.32" width="0.1524" layer="91"/>
+<wire x1="462.28" y1="147.32" x2="457.2" y2="147.32" width="0.1524" layer="91"/>
 <pinref part="R64" gate="G$1" pin="2"/>
 <junction x="462.28" y="147.32"/>
@@
 <pinref part="IC5" gate="G$1" pin="FB"/>
 <pinref part="R72" gate="G$1" pin="1"/>
-<wire x1="454.66" y1="132.08" x2="487.68" y2="132.08" width="0.1524" layer="91"/>
+<wire x1="457.2" y1="132.08" x2="487.68" y2="132.08" width="0.1524" layer="91"/>
 <pinref part="R71" gate="G$1" pin="2"/>
 <wire x1="487.68" y1="137.16" x2="487.68" y2="132.08" width="0.1524" layer="91"/>
@@
 <segment>
 <pinref part="IC5" gate="G$1" pin="BST"/>
-<wire x1="454.66" y1="157.48" x2="457.2" y2="157.48" width="0.1524" layer="91"/>
 <wire x1="457.2" y1="157.48" x2="457.2" y2="160.02" width="0.1524" layer="91"/>
 <pinref part="C36" gate="G$1" pin="1"/>
@@
 </segment>
 <segment>
-<pinref part="IC1" gate="G$1" pin="PD2(OC0C/RXD0)"/>
-<wire x1="48.26" y1="271.78" x2="7.62" y2="271.78" width="0.1524" layer="91"/>
-<label x="7.62" y="271.78" size="1.778" layer="95"/>
-</segment>
-</net>
+<pinref part="IC1" gate="G$1" pin="PE2(OC0C/RXD0)"/>
+<wire x1="48.26" y1="246.38" x2="10.16" y2="246.38" width="0.1524" layer="91"/>
+<label x="10.16" y="246.38" size="1.778" layer="95"/>
+</segment>
+</net>

Commit message: few changes on board
Parts:
- added R74, R75: 270-E, robotter_resistor:270-E
- R29, R34: value 4K7-E -> 8K2-E; device robotter_resistor:4K7-E -> robotter_resistor:8K2-E
- R36, R41: value nc -> 3K09-F; device rcl:R-EU_R0603 -> robotter_resistor:3K09-F
Connections:
- net +3V3: now also R74.2, R75.2
- net IR_SENSOR_0_OUTPUT_3V3: now also R74.1
- net IR_SENSOR_1_OUTPUT_3V3: now also R75.1
Other:
- note added: "connector to IR sensor : S15-PA-2-A00-PK or S15-PA-2-A00-NK"
- moved on the sheet: R34, R36
Changed lines of the file:
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@@
 <part name="GND64" library="supply1" deviceset="GND" device=""/>
 <part name="D4" library="robotter_diode" deviceset="BZV55-C3V3" device="SOD80C" value="bzv55-c3v3"/>
-<part name="R41" library="rcl" deviceset="R-EU_" device="R0603" value="nc"/>
+<part name="R41" library="robotter_resistor" deviceset="3K09" device="-F" value="3K09-F"/>
 <part name="IR_SENSOR1" library="robotter_connector" deviceset="794618-4" device=""/>
 <part name="GND71" library="supply1" deviceset="GND" device=""/>
@@
 <part name="FRAME2" library="frames" deviceset="A4L-LOC" device=""/>
 <part name="D3" library="robotter_diode" deviceset="BZV55-C3V3" device="SOD80C" value="bzv55-c3v3"/>
-<part name="R36" library="rcl" deviceset="R-EU_" device="R0603" value="nc"/>
+<part name="R36" library="robotter_resistor" deviceset="3K09" device="-F" value="3K09-F"/>
 <part name="R27" library="rcl" deviceset="R-EU_" device="R0603" value="nc"/>
 <part name="GND13" library="supply1" deviceset="GND" device=""/>
@@
 <part name="T5" library="robotter_ic" deviceset="NTGS4111" device="PT1G" value="NTGS4111PT1G"/>
 <part name="T2" library="robotter_ic" deviceset="NTGS4111" device="PT1G" value="NTGS4111PT1G"/>
-<part name="R34" library="robotter_resistor" deviceset="4K7" device="-E"/>
-<part name="R29" library="robotter_resistor" deviceset="4K7" device="-E"/>
+<part name="R34" library="robotter_resistor" deviceset="8K2" device="-E"/>
+<part name="R29" library="robotter_resistor" deviceset="8K2" device="-E"/>
 <part name="IC4" library="robotter_ic" deviceset="74LVC4245" device="APW"/>
 <part name="P+4" library="supply1" deviceset="+5V" device=""/>
@@
 <part name="IDX0" library="robotter_others" deviceset="PRISM_INDEX_EXTENSION" device="_MALE"/>
 <part name="GND9" library="supply1" deviceset="GND" device=""/>
+<part name="R74" library="robotter_resistor" deviceset="270" device="-E"/>
+<part name="R75" library="robotter_resistor" deviceset="270" device="-E"/>
+<part name="+3V12" library="supply1" deviceset="+3V3" device=""/>
+<part name="+3V13" library="supply1" deviceset="+3V3" device=""/>
 </parts>
 <sheets>
@@
 <text x="279.4" y="-167.64" size="1.778" layer="91">led used to show idx activity</text>
 <text x="492.76" y="162.56" size="1.778" layer="91">3,3V 1A</text>
+<text x="86.36" y="81.28" size="1.778" layer="91">connector to IR sensor :
+S15-PA-2-A00-PK
+or
+S15-PA-2-A00-NK</text>
+<text x="86.36" y="-114.3" size="1.778" layer="91">connector to IR sensor :
+S15-PA-2-A00-PK
+or
+S15-PA-2-A00-NK</text>
 </plain>
 <instances>
@@
 <instance part="FRAME2" gate="G$1" x="0" y="-185.42"/>
 <instance part="D3" gate="G$1" x="154.94" y="99.06" rot="R90"/>
-<instance part="R36" gate="G$1" x="162.56" y="101.6" rot="R90"/>
+<instance part="R36" gate="G$1" x="165.1" y="101.6" rot="R90"/>
 <instance part="R27" gate="G$1" x="137.16" y="101.6" rot="R90"/>
 <instance part="GND13" gate="1" x="86.36" y="38.1" smashed="yes">
@@
 <instance part="T5" gate="G$1" x="91.44" y="127" rot="R90"/>
 <instance part="T2" gate="G$1" x="83.82" y="-71.12" rot="R90"/>
-<instance part="R34" gate="G$1" x="167.64" y="-91.44"/>
+<instance part="R34" gate="G$1" x="165.1" y="-91.44"/>
 <instance part="R29" gate="G$1" x="147.32" y="106.68"/>
 <instance part="IC4" gate="G$1" x="444.5" y="243.84"/>
@@
 <instance part="IDX0" gate="G$1" x="195.58" y="147.32"/>
 <instance part="GND9" gate="1" x="7.62" y="332.74"/>
+<instance part="R74" gate="G$1" x="154.94" y="111.76" rot="R90"/>
+<instance part="R75" gate="G$1" x="172.72" y="-86.36" rot="R90"/>
+<instance part="+3V12" gate="G$1" x="154.94" y="119.38"/>
+<instance part="+3V13" gate="G$1" x="172.72" y="-78.74"/>
 </instances>
 <busses>
@@
 <pinref part="R23" gate="G$1" pin="1"/>
 <wire x1="104.14" y1="91.44" x2="119.38" y2="91.44" width="0.1524" layer="91"/>
-<wire x1="162.56" y1="96.52" x2="162.56" y2="91.44" width="0.1524" layer="91"/>
+<wire x1="165.1" y1="96.52" x2="165.1" y2="91.44" width="0.1524" layer="91"/>
 <pinref part="R36" gate="G$1" pin="1"/>
 <pinref part="D3" gate="G$1" pin="A"/>
@@
 <wire x1="137.16" y1="91.44" x2="137.16" y2="96.52" width="0.1524" layer="91"/>
 <wire x1="137.16" y1="91.44" x2="154.94" y2="91.44" width="0.1524" layer="91"/>
-<wire x1="154.94" y1="91.44" x2="162.56" y2="91.44" width="0.1524" layer="91"/>
+<wire x1="154.94" y1="91.44" x2="165.1" y2="91.44" width="0.1524" layer="91"/>
 <junction x="119.38" y="91.44"/>
 <junction x="104.14" y="91.44"/>
@@
 <wire x1="467.36" y1="-22.86" x2="467.36" y2="-30.48" width="0.1524" layer="91"/>
 </segment>
+<segment>
+<pinref part="R74" gate="G$1" pin="2"/>
+<pinref part="+3V12" gate="G$1" pin="+3V3"/>
+</segment>
+<segment>
+<pinref part="R75" gate="G$1" pin="2"/>
+<pinref part="+3V13" gate="G$1" pin="+3V3"/>
+</segment>
 </net>
 <net name="/RESET_3V3" class="0">
@@
 <segment>
 <wire x1="187.96" y1="-91.44" x2="205.74" y2="-91.44" width="0.1524" layer="91"/>
+<wire x1="170.18" y1="-91.44" x2="172.72" y2="-91.44" width="0.1524" layer="91"/>
 <wire x1="172.72" y1="-91.44" x2="175.26" y2="-91.44" width="0.1524" layer="91"/>
 <wire x1="175.26" y1="-91.44" x2="187.96" y2="-91.44" width="0.1524" layer="91"/>
@@
 <pinref part="D4" gate="G$1" pin="C"/>
 <pinref part="R34" gate="G$1" pin="2"/>
+<pinref part="R75" gate="G$1" pin="1"/>
+<junction x="172.72" y="-91.44"/>
 </segment>
 <segment>
@@
 <pinref part="IR_SENSOR1" gate="G$1" pin="2"/>
 <pinref part="R21" gate="G$1" pin="2"/>
-<wire x1="162.56" y1="-91.44" x2="121.92" y2="-91.44" width="0.1524" layer="91"/>
+<wire x1="160.02" y1="-91.44" x2="121.92" y2="-91.44" width="0.1524" layer="91"/>
 <pinref part="R20" gate="G$1" pin="1"/>
 <pinref part="R34" gate="G$1" pin="1"/>
@@
 <net name="IR_SENSOR_0_OUTPUT_3V3" class="0">
 <segment>
-<wire x1="162.56" y1="106.68" x2="182.88" y2="106.68" width="0.1524" layer="91"/>
+<wire x1="165.1" y1="106.68" x2="182.88" y2="106.68" width="0.1524" layer="91"/>
 <wire x1="152.4" y1="106.68" x2="154.94" y2="106.68" width="0.1524" layer="91"/>
-<wire x1="154.94" y1="106.68" x2="162.56" y2="106.68" width="0.1524" layer="91"/>
+<wire x1="154.94" y1="106.68" x2="165.1" y2="106.68" width="0.1524" layer="91"/>
 <wire x1="154.94" y1="101.6" x2="154.94" y2="106.68" width="0.1524" layer="91"/>
-<junction x="162.56" y="106.68"/>
+<junction x="165.1" y="106.68"/>
 <junction x="154.94" y="106.68"/>
 <label x="167.64" y="106.68" size="1.778" layer="95"/>
@@
 <pinref part="D3" gate="G$1" pin="C"/>
 <pinref part="R29" gate="G$1" pin="2"/>
-</segment>
-<segment>
+<pinref part="R74" gate="G$1" pin="1"/>
+</segment>
+<segment>

Commit message: mouser component ref added
Parts:
- IC6: device linear:NCV78M05BDTRKG -> robotter_ic:NCV78M05BDTRKG
- MOT0, MOT1: device con-molex:22-27-2021-02 -> robotter_connector:22-27-2021-02
Changed lines of the file:
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@@
 <part name="GND4" library="supply1" deviceset="GND" device=""/>
 <part name="H2" library="holes" deviceset="MOUNT-PAD-ROUND" device="5.5"/>
-<part name="MOT1" library="con-molex" deviceset="22-?-02" device="27-2021"/>
+<part name="MOT1" library="robotter_connector" deviceset="22-?-02" device="27-2021"/>
 <part name="D1" library="robotter_diode" deviceset="CGRM400*-G" device="" technology="4"/>
 <part name="FRAME2" library="frames" deviceset="A4L-LOC" device=""/>
@@
 <part name="GND24" library="supply1" deviceset="GND" device=""/>
 <part name="GND25" library="supply1" deviceset="GND" device=""/>
-<part name="IC6" library="linear" deviceset="NCV78M" device="" technology="05BDTRKG"/>
+<part name="IC6" library="robotter_ic" deviceset="NCV78M" device="" technology="05BDTRKG"/>
 <part name="C32" library="robotter_capacitor" deviceset="10UF" device="-C_25V" value="10µF 25V"/>
 <part name="C37" library="robotter_capacitor" deviceset="10UF" device="-C_25V" value="10µF 25V"/>
@@
 <part name="R22" library="robotter_resistor" deviceset="0" device="-F"/>
 <part name="R23" library="robotter_resistor" deviceset="0" device="-F"/>
-<part name="MOT0" library="con-molex" deviceset="22-?-02" device="27-2021"/>
+<part name="MOT0" library="robotter_connector" deviceset="22-?-02" device="27-2021"/>
 <part name="L1" library="robotter_inductor" deviceset="FERRITE_220OHMS" device="" value="220 ohms"/>
 <part name="R1" library="robotter_resistor" deviceset="0" device="-E"/>

Commit message: added assembly variant to board
Other:
- note added: "MASTER NRF24L01"
- note added: "MASTER XBEE"
- note added: "MASTER XBEE / NRF24L01"
Changed lines of the file:
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@@
 </attributes>
 <variantdefs>
+<variantdef name="Master Xbee"/>
+<variantdef name="Slave"/>
 </variantdefs>
 <classes>
@@
 <part name="LK3" library="robotter_diode" deviceset="LED_" device="G"/>
 <part name="GND17" library="supply1" deviceset="GND" device=""/>
-<part name="XB1" library="robotter_ic" deviceset="XBEE" device="-PRO"/>
+<part name="XB1" library="robotter_ic" deviceset="XBEE" device="-PRO">
+<variant name="Slave" populate="no"/>
+</part>
 <part name="BAL1" library="robotter_connector" deviceset="794618-8" device=""/>
 <part name="BAL2" library="robotter_connector" deviceset="794618-8" device=""/>
@@
 <part name="GND18" library="supply1" deviceset="GND" device=""/>
 <part name="GND21" library="supply1" deviceset="GND" device=""/>
-<part name="BATT" library="robotter_connector" deviceset="1445055-2" device=""/>
-<part name="D5" library="robotter_diode" deviceset="50WQ03" device=""/>
+<part name="BATT" library="robotter_connector" deviceset="1445055-2" device="">
+<variant name="Master Xbee" populate="no"/>
+<variant name="Slave" populate="no"/>
+</part>
+<part name="D5" library="robotter_diode" deviceset="50WQ03" device="">
+<variant name="Slave" populate="no"/>
+</part>
 <part name="GND23" library="supply1" deviceset="GND" device=""/>
-<part name="SW_BATT" library="robotter_others" deviceset="2MS1T2B4M6QNS" device=""/>
+<part name="SW_BATT" library="robotter_others" deviceset="2MS1T2B4M6QNS" device="">
+<variant name="Slave" populate="no"/>
+</part>
 <part name="T7" library="robotter_ic" deviceset="*-NPN-" device="SOT23-BEC" technology="MMBT2222ALT1" value="MMBT2222LT1G"/>
-<part name="R51" library="robotter_resistor" deviceset="1K" device="-F"/>
-<part name="R46" library="robotter_resistor" deviceset="10K" device="-E"/>
+<part name="R51" library="robotter_resistor" deviceset="1K" device="-F">
+<variant name="Slave" populate="no"/>
+</part>
+<part name="R46" library="robotter_resistor" deviceset="10K" device="-E">
+<variant name="Slave" populate="no"/>
+</part>
 <part name="RF" library="robotter_diode" deviceset="LED_" device="Y" value="YELLOW"/>
 <part name="R28" library="robotter_resistor" deviceset="270" device="-F"/>
@@
 <part name="R30" library="robotter_resistor" deviceset="10K" device="-F"/>
 <part name="R33" library="robotter_resistor" deviceset="10K" device="-F"/>
-<part name="R55" library="robotter_resistor" deviceset="10K" device="-F"/>
-<part name="R54" library="robotter_resistor" deviceset="10K" device="-F"/>
+<part name="R55" library="robotter_resistor" deviceset="10K" device="-F">
+<variant name="Slave" populate="no"/>
+</part>
+<part name="R54" library="robotter_resistor" deviceset="10K" device="-F">
+<variant name="Slave" populate="no"/>
+</part>
 <part name="R20" library="robotter_resistor" deviceset="10K" device="-F"/>
 <part name="R9" library="robotter_resistor" deviceset="10K" device="-F"/>
@@
 <part name="R15" library="robotter_resistor" deviceset="10K" device="-F"/>
 <part name="R14" library="robotter_resistor" deviceset="10K" device="-F"/>
-<part name="C20" library="robotter_capacitor" deviceset="10UF" device="-C_25V" value="10µF 25V"/>
-<part name="C21" library="robotter_capacitor" deviceset="10UF" device="-C_25V" value="10µF 25V"/>
-<part name="C23" library="robotter_capacitor" deviceset="100NF" device="-F" value="100nF 50V"/>
+<part name="C20" library="robotter_capacitor" deviceset="10UF" device="-C_25V" value="10µF 25V">
+<variant name="Slave" populate="no"/>
+</part>
+<part name="C21" library="robotter_capacitor" deviceset="10UF" device="-C_25V" value="10µF 25V">
+<variant name="Slave" populate="no"/>
+</part>
+<part name="C23" library="robotter_capacitor" deviceset="100NF" device="-F" value="100nF 50V">
+<variant name="Slave" populate="no"/>
+</part>
 <part name="C34" library="robotter_capacitor" deviceset="100NF" device="-F" value="100nF 50V"/>
 <part name="C35" library="robotter_capacitor" deviceset="100NF" device="-F" value="100nF 50V"/>
@@
 <part name="R61" library="robotter_resistor" deviceset="1K" device="-E" value="1k"/>
 <part name="C24" library="robotter_capacitor" deviceset="330UF" device="" value="330µF 35V"/>
-<part name="T8" library="robotter_ic" deviceset="NTGS4111" device="PT1G" value="NTGS4111PT1G"/>
+<part name="T8" library="robotter_ic" deviceset="NTGS4111" device="PT1G" value="NTGS4111PT1G">
+<variant name="Slave" populate="no"/>
+</part>
 <part name="T5" library="robotter_ic" deviceset="NTGS4111" device="PT1G" value="NTGS4111PT1G"/>
 <part name="T2" library="robotter_ic" deviceset="NTGS4111" device="PT1G" value="NTGS4111PT1G"/>
@@
 <part name="R4" library="robotter_resistor" deviceset="0" device="-E"/>
 <part name="GND6" library="supply1" deviceset="GND" device=""/>
-<part name="IC7" library="robotter_ic" deviceset="NRF24L01+" device=""/>
+<part name="IC7" library="robotter_ic" deviceset="NRF24L01+" device="">
+<variant name="Master Xbee" populate="no"/>
+<variant name="Slave" populate="no"/>
+</part>
 <part name="+3V10" library="supply1" deviceset="+3V3" device=""/>
 <part name="GND7" library="supply1" deviceset="GND" device=""/>
-<part name="C27" library="robotter_capacitor" deviceset="10UF" device="-C_25V" value="10µF 25V"/>
-<part name="C30" library="robotter_capacitor" deviceset="100NF" device="-F" value="100nF 50V"/>
-<part name="R67" library="robotter_resistor" deviceset="10K" device="-F"/>
+<part name="C27" library="robotter_capacitor" deviceset="10UF" device="-C_25V" value="10µF 25V">
+<variant name="Master Xbee" populate="no"/>
+<variant name="Slave" populate="no"/>
+</part>
+<part name="C30" library="robotter_capacitor" deviceset="100NF" device="-F" value="100nF 50V">
+<variant name="Master Xbee" populate="no"/>
+<variant name="Slave" populate="no"/>
+</part>
+<part name="R67" library="robotter_resistor" deviceset="10K" device="-F">
+<variant name="Master Xbee" populate="no"/>
+<variant name="Slave" populate="no"/>
+</part>
 <part name="GND8" library="supply1" deviceset="GND" device=""/>
-<part name="R43" library="robotter_resistor" deviceset="10K" device="-F"/>
-<part name="R42" library="robotter_resistor" deviceset="10K" device="-F"/>
+<part name="R43" library="robotter_resistor" deviceset="10K" device="-F">
+<variant name="Slave" populate="no"/>
+</part>
+<part name="R42" library="robotter_resistor" deviceset="10K" device="-F">
+<variant name="Slave" populate="no"/>
+</part>
 <part name="IDX0" library="robotter_others" deviceset="PRISM_INDEX_EXTENSION" device="_MALE"/>
 <part name="GND9" library="supply1" deviceset="GND" device=""/>
@@
 <text x="210.82" y="320.04" size="1.778" layer="91">use internal pullup of atxmega
 to read beacon id</text>
-<text x="292.1" y="96.52" size="1.778" layer="91">SW_BATT is a switch used to drive the mos that cut power</text>
+<text x="292.1" y="101.6" size="1.778" layer="91">SW_BATT is a switch used to drive the mos that cut power</text>
 <text x="279.4" y="-167.64" size="1.778" layer="91">led used to show idx activity</text>
 <text x="492.76" y="162.56" size="1.778" layer="91">3,3V 1A</text>
@@
 or
 S15-PA-2-A00-NK</text>
-<text x="86.36" y="-114.3" size="1.778" layer="91">connector to IR sensor :
+<text x="86.36" y="-116.84" size="1.778" layer="91">connector to IR sensor :
 S15-PA-2-A00-PK
 or
 S15-PA-2-A00-NK</text>
+<wire x1="274.32" y1="66.04" x2="337.82" y2="66.04" width="1.27" layer="97" style="longdash"/>
+<wire x1="337.82" y1="66.04" x2="337.82" y2="170.18" width="1.27" layer="97" style="longdash"/>
+<wire x1="337.82" y1="170.18" x2="274.32" y2="170.18" width="1.27" layer="97" style="longdash"/>
+<wire x1="274.32" y1="170.18" x2="274.32" y2="66.04" width="1.27" layer="97" style="longdash"/>
+<wire x1="271.78" y1="-96.52" x2="271.78" y2="-12.7" width="1.27" layer="97" style="longdash"/>
+<wire x1="271.78" y1="-12.7" x2="381" y2="-12.7" width="1.27" layer="97" style="longdash"/>
+<wire x1="381" y1="-12.7" x2="513.08" y2="-12.7" width="1.27" layer="97" style="longdash"/>
+<wire x1="513.08" y1="-12.7" x2="513.08" y2="-96.52" width="1.27" layer="97" style="longdash"/>
+<wire x1="513.08" y1="-96.52" x2="381" y2="-96.52" width="1.27" layer="97" style="longdash"/>
+<text x="274.32" y="-93.98" size="2.54" layer="97">MASTER XBEE</text>
+<text x="386.08" y="-93.98" size="2.54" layer="97">MASTER NRF24L01</text>
+<wire x1="381" y1="-96.52" x2="271.78" y2="-96.52" width="1.27" layer="97" style="longdash"/>
+<wire x1="381" y1="-96.52" x2="381" y2="-12.7" width="1.27" layer="97" style="longdash"/>
+<text x="279.4" y="71.12" size="2.54" layer="97">MASTER XBEE / NRF24L01</text>
 </plain>
 <instances>

Commit message: prism v2 : modifications after beacon integration : mirror motor supplied by vbat or +15V, diode B160 pinout corrected
Parts:
- added R76, R77, R78, R79: 0-E, robotter_resistor:0-E
Connections:
- new net VCC_MOT0: C7.1, D2.C, MOT0-2.S, R76.2, R77.2
- new net VCC_MOT1: C6.1, D1.C, MOT1-2.S, R78.2, R79.2
- net +15V: now also R77.1, R78.1
- net VBAT: now also R76.1, R79.1; no longer C6.1, C7.1, D1.C, D2.C, MOT0-2.S, MOT1-2.S
Other:
- note added: "NC if S15-PA-2-A00-NK"
- note added: "WARNING : B160 diode has inverted footprint !"
- note added: "master : R1 NC, R2 NC, R4 NC slave 1: R1 0, R2 NC, R4 0 slave 2: R1 NC, R2 NC, R4 0"
- moved on the sheet: R74, R75
