File: hardware/prism/prism.brd (EAGLE design)
At the start: 100 x 80 mm, 136 parts, among them IC1 MAX3232CSE, IC2 XMEGA128-A1, IC3 LM1086CS-3.3, J1 1445055-2, J2 2MS1T2B4M6QNS, K1 LED_G, K2 LED_G, K3 LED_G, K4 LED_G, K5 LED_G, K6 LED_G, K7 LED_G, K8 LED_G, T1 FDFS2P753Z, T2 MMBT2222LT1G, T3 MMBT2222LT1G, T4 FDFS2P753Z, T5 MMBT2222LT1G, T6 MMBT2222LT1G, T7 FDFS2P753Z, T8 MMBT2222LT1G

Commit message: add 3,3v and 5v regulator
Parts:
- added C30: 1µF 25V, robotter_capacitor:C1206
- added C31: 10nF 50V, robotter_capacitor:C0603
- added C32: 100nF 50V, robotter_capacitor:C0603
- added C33, C34: 10µF 25V, robotter_capacitor:C1210
- added D8: B160-13F, robotter_diode:SMA
- added IC4: LM25011MY, robotter_ic:MSOP10_THERMAL
- added L1: SDR0805-270KL, robotter_inductor:SDR0805
- added R58: 75K-F, robotter_resistor:R0603
- added R59: 100_1W-1W, robotter_resistor:0309/12
- added R60: 10K-F, robotter_resistor:R0603
- added R61: 3K09-F, robotter_resistor:R0603
- C19, C23, C25, C26: device rcl:C0805 -> robotter_capacitor:C0603
- C21: value C_10UF -> 10µF 25V
- C22: value C_10UF -> 1µF 25V; device robotter_capacitor:C1210 -> robotter_capacitor:C1206
- C28: value 10UFC -> 10UF-C_25V
- D7: value 50WQ03 -> (none)
- IC3: value LM1086CS-3.3 -> NCV78M05BDTRKG; device robotter_ic:TO263 -> linear:DPACK_3
- R22: value RES_0 -> 0.27-F; device robotter_resistor:R0805 -> robotter_resistor:R0603
- R27, R31, R38, R45: device rcl:R0603 -> robotter_resistor:R0603
- RF: value YELLOW_0805 -> YELLOW
- T2, T3, T5, T6, T8: device transistor-neu-to92:SOT23-BEC -> robotter_ic:SOT23-BEC
- moved C21 456.3 mm to (-207.0, -355.6)
- moved R22 436.6 mm to (-196.8, -322.6)
- moved R27 410.3 mm to (-186.7, -262.9)
- moved R31 407.1 mm to (-186.7, -268.0)
- moved IC3 385.8 mm to (-204.5, -339.1)
- moved C22 376.5 mm to (-185.4, -284.5)
- moved R38 243.8 mm to (-186.7, -273.1)
- moved R45 237.7 mm to (-186.7, -278.1)
Connections:
- removed net 3V3_BUS: R22.1
- new net N$38: C32.2, D8.A, IC4.9, L1.1
- new net N$39: D8.C, IC4.8, R22.2
- new net N$40: IC4.2, R58.1
- new net N$41: C21.1, IC3.1, R59.2
- new net N$43: C31.1, IC4.4
- new net N$44: IC4.6, R60.1, R61.2
- new net N$48: C32.1, IC4.10
- net +3V3: now also C33.1, L1.2, R61.1; no longer C22.1, IC3.2, IC3.4, R22.2
- net +5V: now also C34.1; no longer C21.1
- net GND: now also C30.2, C31.2, C33.2, C34.2, IC3.4, IC4.5, IC4.7, R22.1, R60.2; no longer IC3.1
- net VBAT: now also C22.1, C30.1, IC4.1, R58.2, R59.1

Commit message: photointerrupter added to board, interfaces added, regulator added
Parts:
- removed D1, D4: bzv55-c3v3, diode:SOD80C
- removed MIRROR_IDX0, MIRROR_IDX1: 794681-4, con-amp:794681-4
- removed R19: nc, rcl:R0603
- removed R20: 4k7, rcl:R0805
- removed R36: nc, rcl:R0805
- removed R47: 10k, rcl:R0603
- removed T7: FDFS2P753Z, robotter:SO8
- added C35, C36, C37, C38, C39, C40: 100nF 50V, robotter_capacitor:C0603
- added IC5, IC6: 74LVC4245A, robotter_ic:TSSOP24
- added PH1, PH2: GP1S58VJ000F, robotter_ic:GP1S58VJ000F
- added R62, R63: 10K-F, robotter_resistor:R0603
- added R64: 4K7-E, robotter_resistor:R0805
- added R65, R66, R67, R68, R69, R70, R71: 0-F, robotter_resistor:R0603
- added T9: NTGS4111PT1G, robotter_ic:TSOP-6
- C1, C10, C11, C12, C13, C14, C15, C16, C3, C4, C5, C6, C7, C9: value C_10UF -> 100nF 50V; device robotter_capacitor:C1210 -> robotter_capacitor:C0603
- C17, C18: value C_10UF -> 15pF_0603_100V; device robotter_capacitor:C1210 -> robotter_capacitor:C0603
- C19, C23, C25, C26: value 100nF -> 100nF 50V
- C2: value 330UF_35V_G_EEEFK1V331P -> 330µF 35V
- C20, C24: value 100nF -> 100nF 50V; device rcl:C0603 -> robotter_capacitor:C0603
- C27: value 10uF_35V_TANTALE -> 10µF 25V; device robotter_capacitor:SMC_D -> robotter_capacitor:C1210
- C28: value 10UF-C_25V -> 10µF 25V
- C29: value 100nF_0603_50V -> 100nF 50V
- C8: value C_10UF -> 10µF 25V
- D2, D5: device diode:SOD80C -> robotter_diode:SOD80C
- D3, D6: device diode:SOD-123_MINI-SMA -> robotter_diode:SOD-123_MINI-SMA
- IR_SENSOR0, IR_SENSOR1: device con-amp:794681-4 -> robotter_connector:794681-4
- R1, R2, R48, R49, R5, R6, R7, R8: value RES_15K -> 270-F; device robotter_resistor:R0805 -> robotter_resistor:R0603
- R12: value nc -> 4K7-F; device rcl:R0603 -> robotter_resistor:R0603
- R13: value 15K_5P_0805 -> 15k 1%
- R14: value 1K_5P_0805 -> 1k
- R15, R23, R24, R26, R3, R30, R32, R35, R37, R39, R4, R40, R46, R51, R52: value 10k -> 10K-F; device rcl:R0603 -> robotter_resistor:R0603
- R16: value 10k -> 4K7-F; device rcl:R0603 -> robotter_resistor:R0603
- R17: value 4k7 -> 270-F; device rcl:R0805 -> robotter_resistor:R0603
- R18: value nc -> 270-F; device rcl:R0805 -> robotter_resistor:R0603
- R43: value 4k7 -> 4K7-E; device rcl:R0805 -> robotter_resistor:R0805
- R44: value 4k7 -> 0-F; device rcl:R0805 -> robotter_resistor:R0603
- T1, T4: value FDFS2P753Z -> NTGS4111PT1G; device robotter:SO8 -> robotter_ic:TSOP-6
- moved R18 904.2 mm to (-221.0, -798.8)
- moved R16 886.8 mm to (-228.6, -768.4)
- moved R17 881.0 mm to (-228.6, -773.4)
- moved R12 769.9 mm to (-228.6, -798.8)
- moved C26 759.6 mm to (-228.6, -788.7)
- moved R15 725.5 mm to (-208.3, -607.1)
- moved C20 701.7 mm to (-208.3, -581.7)
- moved C23 694.4 mm to (-208.3, -586.7)
- moved T1 687.4 mm to (-222.2, -638.8)
- moved C19 685.5 mm to (-208.3, -576.6)
- moved C18 675.8 mm to (-208.3, -571.5)
- moved C17 675.7 mm to (-208.3, -566.4)
- moved R44 664.9 mm to (-228.6, -688.3)
- moved C15 647.6 mm to (-208.3, -543.6)
- moved C16 647.5 mm to (-208.3, -548.6)
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Connections:
- removed net INT1_5V: BAL0.6
- removed net MIRROR_1_INDEX_3V3: D4.C, R12.2, R43.1
- removed net MIRROR_INDEX_0_24V: MIRROR_IDX0.2, R16.1, R17.2, R18.2
- removed net MIRROR_INDEX_1_24V: MIRROR_IDX1.2, R36.2, R37.1, R43.2
- new net INT0_0_3V3: IC6.16, R71.1
- new net INT0_1_3V3: IC6.17, R70.1
- new net INT1_0_3V3: IC6.18, R69.1
- new net INT1_0_5V: BAL0.6, IC5.6, R65.2
- new net INT1_1_3V3: IC6.19, R68.1
- new net MIRROR_INDEX_1_3V3: PH2.TRANSISTOR_C, R12.1
- new net N$47: IC6.5, R44.1
- new net N$49: IC5.19, R68.2
- new net N$50: IC5.17, R70.2
- new net N$51: IC5.18, R69.2
- new net N$52: IC5.16, R71.2
- new net N$53: IC6.6, R65.1
- new net N$54: IC6.8, R67.1
- new net N$55: IC6.7, R66.1
- new net N$56: PH2.LED_A, R18.1
- new net N$57: PH1.LED_A, R17.1
- new net SYNC_IN_0_3V3: IC5.15
- new net SYNC_IN_1_3V3: IC5.14
- new net SYNC_OUT_0_3V3: IC6.15
- new net SYNC_OUT_1_3V3: IC6.14
- net +3V3: now also C19.1, C26.1, C27.1, C35.1, C37.1, C39.1, C40.1, C6.1, IC5.2, IC5.23, IC5.24, IC6.23, IC6.24, R12.2, R16.2, R17.2, R18.2, R62.1, R63.1; no longer C1.1, C27.+
- net +5V: now also C36.1, C38.1, IC5.1, IC6.1
- net GND: now also C17.2, C18.2, C27.2, C3.2, C35.2, C36.2, C37.2, C38.2, C39.2, C40.2, C6.2, IC5.11, IC5.12, IC5.13, IC5.22, IC6.11, IC6.12, IC6.13, IC6.2, IC6.22, PH1.LED_C, PH1.TRANSISTOR_E, PH2.LED_C, PH2.TRANSISTOR_E, R35.1, R37.1; no longer C17.1, C18.1, C27.-, C4.2, C5.2, D1.A, D4.A, MIRROR_IDX0.1, MIRROR_IDX1.1, R12.1, R18.1, R19.1, R36.1, R46.1, R47.1
- net INT0_0_5V: now also IC5.8, R67.2
- net INT0_1_5V: now also IC5.7, R66.2
- net INT1_1_5V: now also IC5.5, R44.2
- net IR_SENSOR_0_OUTPUT_24V: now also R23.1, R64.1; no longer R20.2, R24.1
- net IR_SENSOR_0_OUTPUT_3V3: now also R64.2; no longer R20.1
- net IR_SENSOR_1_OUTPUT_24V: now also R39.1, R43.1; no longer R35.1, R44.2
- net IR_SENSOR_1_OUTPUT_3V3: now also R43.2; no longer R44.1
- net MIRROR_INDEX_0_3V3: now also PH1.TRANSISTOR_C, R16.1; no longer D1.C, R17.1, R19.2
- net MOTOR_PWM_1_3V3: now also R37.2; no longer R46.2
- net N$1: now also C5.1; no longer C3.1
- net N$11: now also C1.1; no longer C4.1
- net N$125: now also R23.2, T1.1, T1.2; no longer R24.2
- net N$128: now also R24.1, T1.3; no longer R23.1, T1.4
- net N$13: now also C3.1; no longer C5.1
- net N$14: now also R46.1, T4.3; no longer R39.1, T4.4
- net N$24: now also C4.2; no longer C6.2
- net N$26: now also R51.2, R52.1, T9.3; no longer R51.1, R52.2, T7.4
- net N$29: now also R51.1; no longer R52.1
- net N$30: now also R52.2, T9.4; no longer R51.2, T7.3
- net N$45: now also C17.1; no longer C17.2
- net N$46: now also C18.1; no longer C18.2
- net N$5: now also C5.2; no longer C3.2
- net N$6: now also C4.1; no longer C6.1
- net N$8: now also C25.1, R39.2, T4.1, T4.2; no longer C24.1, R35.2
- net ON/OFF_SENSOR_1_3V3: now also R35.2; no longer R47.2
- net RX_1_3V3: now also R62.2
- net SYNC_IN_0_5V: now also IC5.9
- net SYNC_IN_1_5V: now also IC5.10
- net SYNC_OUT_0_5V: now also IC6.9
- net SYNC_OUT_1_5V: now also IC6.10
- net TX_1_3V3: now also R63.2
- net VBAT: now also C24.1, R24.2, R46.2, T1.4, T4.4, T9.1, T9.2, T9.5, T9.6; no longer C19.1, C25.1, C26.1, MIRROR_IDX0.3, MIRROR_IDX1.3, R16.2, R23.2, R37.2, R39.2, T1.3, T4.3, T7.5, T7.6
- net XBEE_CTS_3V3: now also IC2.57
- net XBEE_RTS_3V3: now also IC2.58

Commit message: correction after Damien review
Parts:
- IC5, IC6: value 74LVC4245A -> 74LVC4245APW
Changed lines of the file:
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@@
 <attribute name="RS" value="223-0528" x="-222.25" y="-664.21" size="1.778" layer="27" display="off"/>
 </element>
-<element name="IC6" library="robotter_ic" package="TSSOP24" value="74LVC4245A" x="-224.79" y="-671.83"/>
+<element name="IC6" library="robotter_ic" package="TSSOP24" value="74LVC4245APW" x="-224.79" y="-671.83">
+<attribute name="RS" value="380-0500" x="-224.79" y="-671.83" size="1.778" layer="27" display="off"/>
+</element>
 <element name="C35" library="robotter_capacitor" package="C0603" value="100nF 50V" x="-228.6" y="-678.18">
 <attribute name="RS" value=" 723-5534 " x="-228.6" y="-678.18" size="1.778" layer="27" display="off"/>
@@
 <element name="R66" library="robotter_resistor" package="R0603" value="0-F" x="-228.6" y="-698.5"/>
 <element name="R67" library="robotter_resistor" package="R0603" value="0-F" x="-228.6" y="-703.58"/>
-<element name="IC5" library="robotter_ic" package="TSSOP24" value="74LVC4245A" x="-224.79" y="-716.28"/>
+<element name="IC5" library="robotter_ic" package="TSSOP24" value="74LVC4245APW" x="-224.79" y="-716.28">
+<attribute name="RS" value="380-0500" x="-224.79" y="-716.28" size="1.778" layer="27" display="off"/>
+</element>
 <element name="C37" library="robotter_capacitor" package="C0603" value="100nF 50V" x="-228.6" y="-722.63">
 <attribute name="RS" value=" 723-5534 " x="-228.6" y="-717.55" size="1.778" layer="27" display="off"/>

Commit message: prism schematic modified, frist routing test
Parts:
- removed C26: 100nF 50V, robotter_capacitor:C0603
- removed H4: MOUNT-PAD-ROUND5.5, holes:5,5-PAD
- removed IR_SENSOR1: 794681-4, robotter_connector:794681-4
- removed J1: 1445055-2, robotter_connector:1445055-2
- removed J2: 2MS1T2B4M6QNS, robotter_others:2MS1T2B4M6QNS
- removed PH2: GP1S58VJ000F, robotter_ic:GP1S58VJ000F
- removed R41: nc, rcl:R0603
- removed R42: 0, rcl:R0603
- removed R59: 100_1W-1W, robotter_resistor:0309/12
- added BATT: 1445055-2, robotter_connector:1445055-2
- added C41: 180pF 50V, robotter_capacitor:C0603
- added C42, C43: 10µF 25V, robotter_capacitor:C1210
- added D1: B120-13-F, robotter_diode:SMB
- added IC7: LM2731XMF, robotter_ic:SOT23-5
- added J3: 794618-4, robotter_connector:794618-4
- added L2: SRR7032-100M, robotter_inductor:SRR7032
- added L3: 220 ohms, robotter_inductor:R0603
- added R19, R36: 10K_1%-F, robotter_resistor:R0603
- added R20: 113K-F, robotter_resistor:R0603
- added SW_BATT: 2MS1T2B4M6QNS, robotter_others:2MS1T2B4M6QNS
- IR_SENSOR0: value 794681-4 -> 794618-4; device robotter_connector:794681-4 -> robotter_connector:794618-4
- PDI_ATMEL: device robotter_connector:ML6 -> robotter_connector:ML6L
- R12: value 4K7-F -> 0-F
- R18: value 270-F -> 0-F
- R50: value 10K-E -> 1K-F; device robotter_resistor:R0805 -> robotter_resistor:R0603
- moved C40 918.0 mm to (97.9, 64.3), flipped to the bottom, turned to 90 degrees
- moved R12 907.0 mm to (90.8, 50.0)
- moved R18 904.3 mm to (87.6, 51.2), turned to 90 degrees
- moved R17 856.5 mm to (23.5, 45.1), flipped to the bottom, turned to 270 degrees
- moved R71 855.1 mm to (60.1, 56.9), turned to 270 degrees
- moved R70 851.0 mm to (62.1, 56.9), turned to 270 degrees
- moved R69 847.0 mm to (64.1, 56.9), turned to 270 degrees
- moved R16 846.0 mm to (20.8, 40.0), flipped to the bottom, turned to 180 degrees
- moved C39 843.2 mm to (20.8, 42.2), flipped to the bottom
- moved R68 842.9 mm to (66.2, 56.9), turned to 270 degrees
- moved PH1 835.3 mm to (21.6, 43.3), turned to 90 degrees
- moved C38 832.2 mm to (66.9, 50.3), turned to 180 degrees
- moved C37 831.3 mm to (66.9, 54.4), turned to 180 degrees
- moved IC5 821.6 mm to (64.4, 52.7), flipped to the bottom
- moved R67 819.0 mm to (58.7, 63.4), turned to 270 degrees
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Connections:
- removed net IR_SENSOR_OUTPUT_0_3V3: IC2.17
- removed net IR_SENSOR_OUTPUT_1_3V3: IC2.37
- removed net MIRROR_INDEX_10_3V3: IC2.38
- removed net N$125: C20.1, IR_SENSOR0.3, R23.2, R25.2, T1.1, T1.2, T1.5, T1.6
- removed net N$15: IR_SENSOR1.4, R41.2, R42.1
- new net +15V: C20.1, C25.1, C41.1, C42.1, D1.C, R20.1, R24.2, R46.2, T1.4, T4.4
- new net N$58: J3.3, R12.2, R39.2, T4.1, T4.2, T4.5, T4.6
- new net N$59: D1.A, IC7.1, L2.2
- new net N$60: C41.2, IC7.3, R19.2, R20.2
- new net N$63: IC7.4, R36.1
- net +3V3: now also L3.2; no longer C26.1, C7.1, C8.1, IC2.4, IC2.94, R12.2, R18.2
- net GND: now also BATT.1, C42.2, C43.2, IC7.2, J3.1, R18.1, R19.1; no longer C26.2, H4.B5,5, IR_SENSOR1.1, J1.1, PH2.LED_C, PH2.TRANSISTOR_E, R41.1
- net IR_SENSOR_0_OUTPUT_3V3: now also IC2.17
- net IR_SENSOR_1_OUTPUT_24V: now also J3.2; no longer IR_SENSOR1.2
- net IR_SENSOR_1_OUTPUT_3V3: now also IC2.37
- net MIRROR_INDEX_1_3V3: now also IC2.38; no longer PH2.TRANSISTOR_C, R12.1
- net N$23: now also BATT.2, SW_BATT.2; no longer J1.2, J2.2
- net N$41: now also J3.4, R12.1, R18.2; no longer C21.1, IC3.1, R59.2
- net N$56: now also IR_SENSOR0.3, R23.2, R25.2, T1.1, T1.2, T1.5, T1.6; no longer PH2.LED_A, R18.1
- net N$8: now also C7.1, C8.1, IC2.4, IC2.94, L3.1; no longer C25.1, IR_SENSOR1.3, R39.2, R42.2, T4.1, T4.2, T4.5, T4.6
- net ON/OFF_SENSOR_1_3V1: now also SW_BATT.1; no longer J2.1
- net SYNC_IN_0_3V3: now also IC2.19
- net SYNC_IN_1_3V3: now also IC2.20
- net SYNC_OUT_0_3V3: now also IC2.21
- net SYNC_OUT_1_3V3: now also IC2.22
- net VBAT: now also C21.1, C43.1, IC3.1, IC7.5, L2.1, R36.2; no longer R24.2, R46.2, R59.1, T1.4, T4.4
Other:
- board size 100 x 80 mm -> 100 x 79 mm
