File: hardware/meca_2014/meca_2014.sch (EAGLE design)
At the start: 128 parts, among them IC1 MAX3232CSE, IC10 74LVC1T45DBV, IC11 74LVC1T45DBV, IC12 LM2596S-ADJ, IC2 XMEGA128-A1, IC3 LM1086CS-3.3, IC4 MPXV5100GC6U, IC5 LM2596S-ADJ, IC6 74LVC4245APW, IC8 MPXV5100GC6U, T1 NTR4503NT1G, T2 NTR4503NT1G

Commit message: meca 2014 : routing done
Connections:
- removed net PWM1: SV7.3
- removed net PWM2: SV6.3
- removed net PWM3: SV1.3
- removed net PWM3_3V3: IC6.IO_VL3
- net +3V3: now also IC11.VCCA
- net +5V: now also IC11.VCCB
- net PWM1_5V: now also SV7.3
- net PWM2_5V: now also SV6.3
- net PWM3_5V: now also SV1.3
- net PWM_C4_3V3: now also IC6.IO_VL3; no longer IC6.IO_VL1
- net PWM_D1_3V3: now also IC6.IO_VL1; no longer IC6.IO_VL2
- net PWM_D2_3V3: now also IC6.IO_VL2
Changed lines of the file:
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@@
 <text x="358.14" y="-43.18" size="1.778" layer="91">Vbatt : 12-26V</text>
 <text x="142.24" y="-264.16" size="1.778" layer="91">analog voltage used to verify that the voltage of the vacuum pump command</text>
-<text x="12.7" y="-134.62" size="1.778" layer="91">renommer les nets une fois la carte routée par pwm_E0_3v3 par exemple, renommer aussi les connecteurs</text>
+<text x="10.16" y="-142.24" size="1.778" layer="91">renommer les nets une fois la carte routée par pwm_E0_3v3 par exemple, renommer aussi les connecteurs</text>
 <text x="193.04" y="-129.54" size="1.778" layer="91">verifier sens transceiver</text>
 <text x="134.62" y="66.04" size="1.778" layer="91">ne pas connecter SS du port sur lequel est connecte la spi du codeur</text>
@@
 <segment>
 <pinref part="+3V4" gate="G$1" pin="+3V3"/>
-<wire x1="205.74" y1="-27.94" x2="205.74" y2="-20.32" width="0.1524" layer="91"/>
 <pinref part="C28" gate="G$1" pin="1"/>
 <wire x1="177.8" y1="-22.86" x2="177.8" y2="-20.32" width="0.1524" layer="91"/>
 <wire x1="177.8" y1="-20.32" x2="205.74" y2="-20.32" width="0.1524" layer="91"/>
+<pinref part="IC11" gate="G$1" pin="VCCA"/>
+<wire x1="205.74" y1="-20.32" x2="205.74" y2="-27.94" width="0.1524" layer="91"/>
 <junction x="205.74" y="-20.32"/>
 </segment>
@@
 <segment>
 <pinref part="P+3" gate="1" pin="+5V"/>
-<wire x1="210.82" y1="-27.94" x2="210.82" y2="-20.32" width="0.1524" layer="91"/>
 <pinref part="C27" gate="G$1" pin="1"/>
 <wire x1="233.68" y1="-20.32" x2="226.06" y2="-20.32" width="0.1524" layer="91"/>
-<junction x="210.82" y="-20.32"/>
 <pinref part="R17" gate="G$1" pin="2"/>
 <wire x1="226.06" y1="-20.32" x2="210.82" y2="-20.32" width="0.1524" layer="91"/>
 <wire x1="226.06" y1="-27.94" x2="226.06" y2="-20.32" width="0.1524" layer="91"/>
 <junction x="226.06" y="-20.32"/>
+<pinref part="IC11" gate="G$1" pin="VCCB"/>
+<wire x1="210.82" y1="-27.94" x2="210.82" y2="-20.32" width="0.1524" layer="91"/>
+<junction x="210.82" y="-20.32"/>
 </segment>
 <segment>
@@
 </segment>
 </net>
-<net name="PWM3_3V3" class="0">
-<segment>
-<wire x1="162.56" y1="-111.76" x2="180.34" y2="-111.76" width="0.1524" layer="91"/>
-<label x="167.64" y="-111.76" size="1.778" layer="95"/>
-<pinref part="IC6" gate="G$1" pin="IO_VL3"/>
-</segment>
-</net>
-<net name="PWM3" class="0">
-<segment>
-<pinref part="SV1" gate="G$1" pin="3"/>
-<wire x1="53.34" y1="-91.44" x2="55.88" y2="-91.44" width="0.1524" layer="91"/>
-<label x="53.34" y="-91.44" size="1.778" layer="95"/>
-</segment>
-</net>
-<net name="PWM2" class="0">
-<segment>
-<pinref part="SV6" gate="G$1" pin="3"/>
-<wire x1="53.34" y1="-76.2" x2="55.88" y2="-76.2" width="0.1524" layer="91"/>
-<label x="53.34" y="-76.2" size="1.778" layer="95"/>
-</segment>
-</net>
-<net name="PWM1" class="0">
-<segment>
-<pinref part="SV7" gate="G$1" pin="3"/>
-<wire x1="53.34" y1="-60.96" x2="55.88" y2="-60.96" width="0.1524" layer="91"/>
-<label x="53.34" y="-60.96" size="1.778" layer="95"/>
-</segment>
-</net>
 <net name="PWM0_5V" class="0">
 <segment>
@@
 <net name="PWM_D1_3V3" class="0">
 <segment>
-<wire x1="162.56" y1="-109.22" x2="180.34" y2="-109.22" width="0.1524" layer="91"/>
-<label x="167.64" y="-109.22" size="1.778" layer="95"/>
-<pinref part="IC6" gate="G$1" pin="IO_VL2"/>
-</segment>
-<segment>
 <pinref part="IC2" gate="G$1" pin="PD1(OC0B/XCK0/SCL)"/>
 <wire x1="40.64" y1="88.9" x2="12.7" y2="88.9" width="0.1524" layer="91"/>
 <label x="12.7" y="88.9" size="1.778" layer="95"/>
 </segment>
-</net>
-<net name="PWM_C4_3V3" class="0">
-<segment>
+<segment>
+<pinref part="IC6" gate="G$1" pin="IO_VL1"/>
 <wire x1="162.56" y1="-106.68" x2="180.34" y2="-106.68" width="0.1524" layer="91"/>
 <label x="167.64" y="-106.68" size="1.778" layer="95"/>
-<pinref part="IC6" gate="G$1" pin="IO_VL1"/>
-</segment>
+</segment>
+</net>
+<net name="PWM_C4_3V3" class="0">
 <segment>
 <pinref part="IC2" gate="G$1" pin="PC4(OC1A/!SS!)"/>
 <wire x1="40.64" y1="106.68" x2="12.7" y2="106.68" width="0.1524" layer="91"/>
 <label x="12.7" y="106.68" size="1.778" layer="95"/>
+</segment>
+<segment>
+<pinref part="IC6" gate="G$1" pin="IO_VL3"/>
+<wire x1="162.56" y1="-111.76" x2="180.34" y2="-111.76" width="0.1524" layer="91"/>
+<label x="167.64" y="-111.76" size="1.778" layer="95"/>
 </segment>
 </net>
@@
 <pinref part="IC6" gate="G$1" pin="IO_VCC1"/>
 </segment>
+<segment>
+<pinref part="SV7" gate="G$1" pin="3"/>
+<wire x1="53.34" y1="-60.96" x2="55.88" y2="-60.96" width="0.1524" layer="91"/>
+<label x="53.34" y="-60.96" size="1.778" layer="95"/>
+</segment>
 </net>
 <net name="PWM2_5V" class="0">
@@
 <pinref part="IC6" gate="G$1" pin="IO_VCC2"/>
 </segment>
+<segment>
+<pinref part="SV6" gate="G$1" pin="3"/>
+<wire x1="53.34" y1="-76.2" x2="55.88" y2="-76.2" width="0.1524" layer="91"/>
+<label x="53.34" y="-76.2" size="1.778" layer="95"/>
+</segment>
 </net>
 <net name="PWM3_5V" class="0">
@@
 <pinref part="IC6" gate="G$1" pin="IO_VCC3"/>
 </segment>
+<segment>
+<pinref part="SV1" gate="G$1" pin="3"/>
+<wire x1="53.34" y1="-91.44" x2="55.88" y2="-91.44" width="0.1524" layer="91"/>
+<label x="53.34" y="-91.44" size="1.778" layer="95"/>
+</segment>
 </net>
 <net name="PWM_D2_3V3" class="0">
@@
 <label x="12.7" y="86.36" size="1.778" layer="95"/>
 </segment>
-</net>
+<segment>
+<pinref part="IC6" gate="G$1" pin="IO_VL2"/>
+<wire x1="162.56" y1="-109.22" x2="180.34" y2="-109.22" width="0.1524" layer="91"/>
+<label x="167.64" y="-109.22" size="1.778" layer="95"/>
+</segment>
+</net>

Commit message: power supply rerouted, board ready to be sent to manufacturer
Parts:
- removed SV1, SV11, SV12, SV13, SV14, SV6, SV7, SV8: (no value), con-lstb:MA03-1
- added C44: 10µF 25V, robotter_capacitor:10UF-C_25V
- added PC0, PC1, PC2, PC3, PWMC4, PWMD0, PWMD1, PWMD2: (no value), con-lstb:MA03-1
- renumbered COM1 to COLOR_SENS, ERROR to ERR, SV10 to ADCB3, SV3 to ADCB0, SV4 to ADCB1, SV9 to ADCB2
Connections:
- net ADC0 renamed ADCB0
- net ADC1 renamed ADCB1
- net ADC2 renamed ADCB2
- net ADC3 renamed ADCB3
- removed net PC0: IC2.PC0(OC0A/SDA), SV11.3
- removed net PC1: IC2.PC1(OC0B/XCK0/SCL), SV12.3
- removed net PC2: IC2.PC2(OC0C/RXD0), SV13.3
- removed net PC3: IC2.PC3(OC0D/TXD0), SV14.3
- removed net PWM0_5V: IC6.IO_VCC0, SV8.3
- removed net PWM1_5V: IC6.IO_VCC1, SV7.3
- removed net PWM2_5V: IC6.IO_VCC2, SV6.3
- removed net PWM3_5V: IC6.IO_VCC3, SV1.3
- new net PC0_3V3: IC2.PC0(OC0A/SDA), PC0.3
- new net PC1_3V3: IC2.PC1(OC0B/XCK0/SCL), PC1.3
- new net PC2_3V3: IC2.PC2(OC0C/RXD0), PC2.3
- new net PC3_3V3: IC2.PC3(OC0D/TXD0), PC3.3
- new net PWM_C4_5V: IC6.IO_VCC3, PWMC4.3
- new net PWM_D0_5V: IC6.IO_VCC0, PWMD0.3
- new net PWM_D1_5V: IC6.IO_VCC1, PWMD1.3
- new net PWM_D2_5V: IC6.IO_VCC2, PWMD2.3
- net +3V3: now also C44.1, PC0.2, PC1.2, PC2.2, PC3.2; no longer SV11.2, SV12.2, SV13.2, SV14.2
- net +5V: now also PWMC4.2, PWMD0.2, PWMD1.2, PWMD2.2; no longer SV1.2, SV6.2, SV7.2, SV8.2
- net GND: now also C44.2, PC0.1, PC1.1, PC2.1, PC3.1, PWMC4.1, PWMD0.1, PWMD1.1, PWMD2.1; no longer SV1.1, SV11.1, SV12.1, SV13.1, SV14.1, SV6.1, SV7.1, SV8.1

Commit message: few changes before fabrication
Parts:
- added C45, C46: 10µF 25V, robotter_capacitor:10UF-C_25V
Connections:
- net GND: now also C45.2, C46.2
- net VACUUM_PUMP_0_VOLTAGE_MONITOR_0-1V: now also C46.1
- net VACUUM_PUMP_1_VOLTAGE_MONITOR_0-1V: now also C45.1
Changed lines of the file:
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@@
 <part name="GND27" library="supply1" deviceset="GND" device=""/>
 <part name="C44" library="robotter_capacitor" deviceset="10UF" device="-C_25V" value="10µF 25V"/>
+<part name="C45" library="robotter_capacitor" deviceset="10UF" device="-C_25V" value="10µF 25V"/>
+<part name="C46" library="robotter_capacitor" deviceset="10UF" device="-C_25V" value="10µF 25V"/>
 </parts>
 <sheets>
@@
 <instance part="GND27" gate="1" x="121.92" y="-93.98"/>
 <instance part="C44" gate="G$1" x="490.22" y="-144.78"/>
+<instance part="C45" gate="G$1" x="203.2" y="-299.72"/>
+<instance part="C46" gate="G$1" x="203.2" y="-246.38"/>
 </instances>
 <busses>
@@
 <wire x1="185.42" y1="-254" x2="185.42" y2="-246.38" width="0.1524" layer="91"/>
 <junction x="185.42" y="-254"/>
+<pinref part="C46" gate="G$1" pin="2"/>
+<wire x1="195.58" y1="-254" x2="203.2" y2="-254" width="0.1524" layer="91"/>
+<wire x1="203.2" y1="-254" x2="203.2" y2="-251.46" width="0.1524" layer="91"/>
+<junction x="195.58" y="-254"/>
 </segment>
 <segment>
@@
 <wire x1="185.42" y1="-307.34" x2="185.42" y2="-299.72" width="0.1524" layer="91"/>
 <junction x="185.42" y="-307.34"/>
+<pinref part="C45" gate="G$1" pin="2"/>
+<wire x1="195.58" y1="-307.34" x2="203.2" y2="-307.34" width="0.1524" layer="91"/>
+<wire x1="203.2" y1="-307.34" x2="203.2" y2="-304.8" width="0.1524" layer="91"/>
+<junction x="195.58" y="-307.34"/>
 </segment>
 <segment>
@@
 <pinref part="R2" gate="G$1" pin="2"/>
 <pinref part="R26" gate="G$1" pin="1"/>
-<wire x1="195.58" y1="-243.84" x2="233.68" y2="-243.84" width="0.1524" layer="91"/>
+<wire x1="195.58" y1="-243.84" x2="203.2" y2="-243.84" width="0.1524" layer="91"/>
 <label x="200.66" y="-243.84" size="1.778" layer="95"/>
 <junction x="195.58" y="-243.84"/>
+<pinref part="C46" gate="G$1" pin="1"/>
+<wire x1="203.2" y1="-243.84" x2="233.68" y2="-243.84" width="0.1524" layer="91"/>
+<junction x="203.2" y="-243.84"/>
 </segment>
 <segment>
@@
 <pinref part="R28" gate="G$1" pin="2"/>
 <pinref part="R29" gate="G$1" pin="1"/>
-<wire x1="195.58" y1="-297.18" x2="233.68" y2="-297.18" width="0.1524" layer="91"/>
+<wire x1="195.58" y1="-297.18" x2="203.2" y2="-297.18" width="0.1524" layer="91"/>
 <label x="200.66" y="-297.18" size="1.778" layer="95"/>
 <junction x="195.58" y="-297.18"/>
-</segment>
-<segment>
+<pinref part="C45" gate="G$1" pin="1"/>
+<wire x1="203.2" y1="-297.18" x2="233.68" y2="-297.18" width="0.1524" layer="91"/>
+<junction x="203.2" y="-297.18"/>
+</segment>
+<segment>

Commit message: mouser component ref added
Parts:
- AEAT_ENCOD: device con-molex:22-23-2061 -> robotter_connector:22-23-2061
- AX12: device con-amp:1445055-3 -> robotter_connector:1445055-3
- PW_BAT: device con-amp:1445055-2 -> robotter_connector:1445055-2
- UART_CAM: device con-molex:22-23-2031 -> robotter_connector:22-23-2031
Changed lines of the file:
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@@
 <part name="C37" library="robotter_capacitor" deviceset="100NF" device="-F"/>
 <part name="R20" library="robotter_resistor" deviceset="10K" device="-F" value="10k"/>
-<part name="AEAT_ENCOD" library="con-molex" deviceset="22-23-2061" device=""/>
+<part name="AEAT_ENCOD" library="robotter_connector" deviceset="22-23-2061" device=""/>
 <part name="C38" library="robotter_capacitor" deviceset="220UF" device="F_35V"/>
 <part name="C39" library="robotter_capacitor" deviceset="220UF" device="F_35V"/>
@@
 <part name="C42" library="robotter_capacitor" deviceset="220UF" device="F_35V"/>
 <part name="C43" library="robotter_capacitor" deviceset="220UF" device="F_35V"/>
-<part name="UART_CAM" library="con-molex" deviceset="22-23-2031" device=""/>
+<part name="UART_CAM" library="robotter_connector" deviceset="22-23-2031" device=""/>
 <part name="ADCB0" library="con-lstb" deviceset="MA03-1" device="">
 <attribute name="MF" value=""/>
@@
 <part name="L1" library="robotter_inductor" deviceset="SRR1280" device="-150" value="15uH"/>
 <part name="L2" library="robotter_inductor" deviceset="33µH" device="-3.3A" value="33uH"/>
-<part name="AX12" library="con-amp" deviceset="1445055-3" device=""/>
-<part name="PW_BAT" library="con-amp" deviceset="1445055-2" device=""/>
+<part name="AX12" library="robotter_connector" deviceset="1445055-3" device=""/>
+<part name="PW_BAT" library="robotter_connector" deviceset="1445055-2" device=""/>
 <part name="GND5" library="supply1" deviceset="GND" device=""/>
 <part name="R27" library="robotter_resistor" deviceset="3K09" device="-F"/>
