File: hardware/prism_idx_support/prism_idx_support.sch (EAGLE design)
At the start: 8 parts

Commit message: text added
Other:
- note added: "R2 must be 1k6"
Changed lines of the file:
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@@
 <sheet>
 <plain>
+<text x="93.98" y="106.68" size="1.778" layer="91">R2 must be 1k6</text>
 </plain>
 <instances>
