File: hardware/R3D2/R3D2.brd (EAGLE design)
At the start: 75 x 75 mm, 81 parts, among them IC1 MAX3232CSE, IC2 XMEGA128-A1, IC3 LM1086CS-3.3, K1 LED_GREEN_0805, K2 LED_GREEN_0805, K3 LED_GREEN_0805, K4 LED_GREEN_0805, T1 FDFS2P753Z, T2 MMBT2222LT1G, T3 MMBT2222LT1G

Commit message: component refs updated
Parts:
- ALIM: device con-molex:6410-04 -> robotter_connector:6410-04
- C1, C10, C11, C12, C13, C14, C15, C16, C2, C21, C22, C3, C4, C5, C6, C7, C8, C9: value C_100NF_50V_0805 -> 100NF-E
- C17, C18: value C_15PF_100V_0805 -> 15PF-E
- C19, C23: device rcl:C0805 -> robotter_capacitor:C0805
- C20: device rcl:C0603 -> robotter_capacitor:C0603
- COM, ERROR, K1, K2, K3, K4, RUN: value LED_GREEN_0805 -> LED_G
- D1, D2: device diode:SOD80C -> robotter_diode:SOD80C
- D3: device diode:SOD-123_MINI-SMA -> robotter_diode:SOD-123_MINI-SMA
- IR_SENSOR, MIRROR_IDX: device con-amp:794681-4 -> robotter_connector:794681-4
- MOT: device con-molex:6410-02 -> robotter_connector:6410-02
- R10, R11, R5, R6, R7, R8, R9: value RES_270_5P_0805 -> 270-E
- R13, R14, R22: value RES_0_5P_0805 -> 0-E
- R15, R16, R23, R24, R25, R26, R27, R3, R30, R31, R32, R4: device rcl:R0603 -> robotter_resistor:R0603
- R17, R20: device rcl:R0805 -> robotter_resistor:R0805
- T1: value FDFS2P753Z -> IRF7205PBF; device robotter:SO8 -> robotter_ic:SO8
- T2, T3: device transistor-neu-to92:SOT23-BEC -> robotter_ic:SOT23-BEC
Connections:
- net +24V: now also T1.1, T1.2
- net N$125: now also T1.7, T1.8
