File: hardware/R3D2/R3D2.sch (EAGLE design)
At the start: 81 parts, among them IC1 MAX3232CSE, IC2 XMEGA128-A1, IC3 LM1086CS-3.3, K1 LED_GREEN_0805, K2 LED_GREEN_0805, K3 LED_GREEN_0805, K4 LED_GREEN_0805, T1 FDFS2P753Z, T2 MMBT2222LT1G, T3 MMBT2222LT1G

Commit message: component refs updated
Parts:
- ALIM: device con-molex:22-27-2041-04 -> robotter_connector:22-27-2041-04
- C1, C10, C11, C12, C13, C14, C15, C16, C2, C21, C22, C3, C4, C5, C6, C7, C8, C9: value C_100NF_50V_0805 -> 100NF-E; device robotter_capacitor:C_100NF_50V_0805 -> robotter_capacitor:100NF-E
- C17, C18: value C_15PF_100V_0805 -> 15PF-E; device robotter_capacitor:C_15PF_100V_0805 -> robotter_capacitor:15PF-E
- C19, C23: device rcl:C-EUC0805 -> robotter_capacitor:100NF-E
- C20: device rcl:C-EUC0603 -> robotter_capacitor:100NF-F
- COM, ERROR, K1, K2, K3, K4, RUN: value LED_GREEN_0805 -> LED_G; device robotter_diode:LED_GREEN_0805 -> robotter_diode:LED_G
- D1, D2: device diode:ZENER-DIODESOD80C -> robotter_diode:BZV55-C3V3SOD80C
- D3: device diode:CGRM4004-G -> robotter_diode:CGRM4004-G
- IR_SENSOR, MIRROR_IDX: device con-amp:794681-4 -> robotter_connector:794681-4
- MOT: device con-molex:22-27-2021-02 -> robotter_connector:22-27-2021-02
- R10, R11, R5, R6, R7, R8, R9: value RES_270_5P_0805 -> 270-E; device robotter_resistor:RES_270_5P_0805 -> robotter_resistor:270-E
- R13, R14, R22: value RES_0_5P_0805 -> 0-E; device robotter_resistor:RES_0_5P_0805 -> robotter_resistor:0-E
- R15, R16, R23, R24, R26, R3, R30, R32, R4: device rcl:R-EU_R0603 -> robotter_resistor:10K-F
- R17, R20: device rcl:R-EU_R0805 -> robotter_resistor:4K7-E
- R25: device rcl:R-EU_R0603 -> robotter_resistor:0-F
- R27, R31: device rcl:R-EU_R0603 -> robotter_resistor:1K-F
- T1: value FDFS2P753Z -> IRF7205PBF; device robotter:FDFS2P753Z -> robotter_ic:IRF7205PBF
- T2, T3: device transistor-neu-to92:MMBT2222ALT1-NPN-SOT23-BEC -> robotter_ic:MMBT2222ALT1-NPN-SOT23-BEC
Connections:
- net +24V: now also T1.S@1, T1.S@2, T1.S@3; no longer T1.S
- net N$125: now also T1.D@1, T1.D@2, T1.D@3, T1.D@4; no longer T1.D, T1.D1
