File: hardware/robot_wiring/robot_wiring.sch (EAGLE design)
At the start: 23 parts

Commit message: galiper wirring : some connectors added, WIP
Parts:
- added U$17, U$18, U$19, U$20, U$21, U$22: 50394-8051, robotter_wiring:50394-8051
- added U$24, U$25, U$27, U$28, U$30, U$31, U$34, U$35, U$36, U$37, U$38, U$39, U$40, U$41, U$42, U$43, U$46, U$47, U$48, U$49, U$50, U$51, U$52, U$53, U$54, U$55, U$58, U$59, U$60, U$61, U$62, U$63, U$64, U$65, U$66, U$67: 08-50-0113, robotter_wiring:08-50-0113
- added U$68, U$69: 215083-4, robotter_wiring:215083-4
- added U$70, U$71, U$72, U$73, U$74, U$75: 1-2178712-6, robotter_wiring:1-2178712-6
Connections:
- net N$13: now also U$24.P$1; no longer U$9.+
- net N$14: now also U$25.P$1; no longer U$9.-
- net N$15: now also U$28.P$1, U$30.P$1; no longer U$8.GND@2, U$9.GND@2
- net N$16: now also U$21.P$1; no longer U$9.LONG_RANGE_LED_3V3
- net N$17: now also U$20.P$1; no longer U$9.LONG_RANGE_SENSOR_OUTPUT_24V
- net N$18: now also U$19.P$1; no longer U$9.SENSOR_SUPPLY_24V
- net N$19: now also U$17.P$1; no longer U$9.SHORT_RANGE_SENSOR_OUTPUT_24V
- net N$20: now also U$18.P$1; no longer U$9.GND@3
- net N$7: now also U$22.P$1; no longer U$9.SHORT_RANGE_LED_3V3
Other:
- moved on the sheet: BATTERY, GENERAL

Commit message: galiper wirring : all connectors added to super unioc, sabotter and R3D2 boards, WIP for meca board
Parts:
- added U$100, U$101, U$102, U$103, U$104, U$105, U$85, U$86, U$87, U$88, U$89, U$90, U$91, U$92, U$93, U$94, U$95, U$96, U$97, U$98, U$99: 1-794610-1, robotter_wiring:1-794610-1
- added U$109, U$110, U$111, U$112, U$113, U$114, U$115, U$116, U$117, U$118, U$121, U$122, U$123, U$124, U$125, U$126, U$127, U$128, U$129, U$130, U$133, U$134, U$135, U$136, U$137, U$138, U$139, U$140, U$141, U$142: 50394-8051, robotter_wiring:50394-8051
Connections:
- net N$1: now also U$97.P$1, U$99.P$1; no longer U$1.+, U$4.+
- net N$10: now also U$104.P$1; no longer U$8.COLOR_SELECT_3V3
- net N$11: now also U$105.P$1; no longer U$8.GND@4
- net N$12: now also U$103.P$1; no longer U$8.STARTING_CORD_3V3
- net N$15: now also U$101.P$1, U$90.P$1, U$93.P$1; no longer U$4.GND, U$5.GND, U$6.GND
- net N$2: now also U$100.P$1, U$98.P$1; no longer U$1.-, U$4.-
- net N$3: now also U$86.P$1, U$87.P$1; no longer U$3.-, U$6.-
- net N$4: now also U$85.P$1, U$88.P$1; no longer U$3.+, U$6.+
- net N$5: now also U$92.P$1, U$96.P$1; no longer U$2.-, U$5.-
- net N$6: now also U$91.P$1, U$95.P$1; no longer U$2.+, U$5.+

Commit message: galiper wirring : meca board added, need to update board version and final meca wirring
Parts:
- removed U$86, U$95, U$96, U$97, U$98: 1-794610-1, robotter_wiring:1-794610-1
- added U$143, U$144: 215083-4, robotter_wiring:215083-4
- added U$145, U$146: 08-50-0113, robotter_wiring:08-50-0113
- added U$155, U$156, U$157, U$158: 1-794610-1, robotter_wiring:1-794610-1
- added U$26: DC_MOTOR, robotter_wiring:DC_MOTOR
- added U$83: MOTOR_CTRL_PW_V3, robotter_wiring:MOTOR_CTRL_PW_V3
- added U$84: 1-2178712-6, robotter_wiring:1-2178712-6
- U$85: value 1-794610-1 -> 1-2178712-6; device robotter_wiring:1-794610-1 -> robotter_wiring:1-2178712-6
Connections:
- removed net N$15: BATTERY.-, U$101.P$1, U$28.P$1, U$30.P$1, U$90.P$1, U$93.P$1
- new net N$25: U$155.P$1, U$26.+
- new net N$26: U$156.P$1, U$26.-
- net GND: now also BATTERY.-, U$101.P$1, U$146.P$1, U$157.P$1, U$28.P$1, U$30.P$1, U$90.P$1, U$93.P$1
- net N$1: now also U$1.+; no longer U$97.P$1
- net N$2: now also U$1.-; no longer U$98.P$1
- net N$3: now also U$3.-; no longer U$86.P$1
- net N$4: now also U$3.+; no longer U$85.P$1
- net N$5: now also U$2.-; no longer U$96.P$1
- net N$6: now also U$2.+; no longer U$95.P$1
Other:
- note added: "MECA"

Commit message: robot schematic components updated
Changed lines of the file:
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@@
 <part name="U$104" library="robotter_wiring" deviceset="1-794610-1" device=""/>
 <part name="U$105" library="robotter_wiring" deviceset="1-794610-1" device=""/>
-<part name="U$106" library="robotter_wiring" deviceset="794616-4" device=""/>
 <part name="U$107" library="robotter_wiring" deviceset="51021-0500" device=""/>
 <part name="U$108" library="robotter_wiring" deviceset="51021-0500" device=""/>
@@
 <part name="U$84" library="robotter_wiring" deviceset="1-2178712-6" device=""/>
 <part name="U$85" library="robotter_wiring" deviceset="1-2178712-6" device=""/>
+<part name="U$86" library="robotter_wiring" deviceset="794616-4" device=""/>
 </parts>
 <sheets>
@@
 <instance part="U$104" gate="G$1" x="-304.8" y="-10.16" rot="R180"/>
 <instance part="U$105" gate="G$1" x="-304.8" y="-12.7" rot="R180"/>
-<instance part="U$106" gate="G$1" x="-297.18" y="-12.7" rot="MR0"/>
 <instance part="U$107" gate="G$1" x="27.94" y="73.66"/>
 <instance part="U$108" gate="G$1" x="78.74" y="78.74" rot="MR0"/>
@@
 <instance part="U$84" gate="G$1" x="-63.5" y="-236.22"/>
 <instance part="U$85" gate="G$1" x="-38.1" y="-236.22" rot="MR0"/>
+<instance part="U$86" gate="G$2" x="-297.18" y="-10.16"/>
 </instances>
 <busses>
