File: hardware/color_proximity_sensor/color_proximity_sensor.sch (EAGLE design)
At the start: 69 parts, among them IC1 TCS37725FN, IC2 APDS-9800-021, IC4 LM25011MY, IC5 ATXMEGA64D4-AU, J1 PDI_ATMEL_WIDTH, Q1 16 MHz, T1 BC847CDXV6T1G, T4 BC847CDXV6T1G

Commit message: color_proximity_sensor : VL53L0X sensor integrated
Parts:
- removed C6: 22µF 10V, robotter_capacitor:22UF-C_10V
- removed C7, C8: 100nF 50V, robotter_capacitor:100NF-F
- removed C9: 1µF 25V, robotter_capacitor:1UFD_25V
- removed IC2: APDS-9800-021, robotter_ic:APDS-9800-021
- removed R7: 15k 1%, robotter_resistor:15K-F
- added C20: 10µF 25V, robotter_capacitor:10UF-C_25V
- added C21: 100nF 50V, robotter_capacitor:100NF-F
- added IC3: VL53L0x, robotter_ic:VL53L0X
- R3, R4: value 22 ohms -> 10K-F; device robotter_resistor:22-F -> robotter_resistor:10K-F
- R5: value 10K-F -> 3K09-F; device robotter_resistor:10K-F -> robotter_resistor:3K09-F
- R6: value 1k -> 3K09-F; device robotter_resistor:1K-F -> robotter_resistor:3K09-F
Connections:
- removed net APDS_AMBIENT_0-300MV: C9.2, IC2.ALS_IOUT, IC5.PA0/ADCA0/AREF, R6.2
- removed net APDS_ENABLE_3V3: IC2.PS_ENB, IC5.\S\S/PD4
- removed net APDS_LED_PWM_3V3: IC2.LEDON, IC5.TXD0/OC0D/PD3
- removed net APDS_OUTPUT_3V3: IC2.PS_DOUT, IC5.MOSI/PD5, R5.1
- removed net APDS_PROXIMITY_ANA_0-0.65V: C8.2, IC2.PS_PFILT, IC5.PA1/ADCA1, R7.2
- removed net N$2: IC2.LEDK, R3.2, R4.2
- new net CE_VL53L0X_3V3: IC3.XSHUT, IC5.MISO/PD6, R3.1
- new net INT_VL53L0X_3V3: IC3.GPIO1, IC5.MOSI/PD5, R4.1
- new net SCL_VL53V0X_3V3: IC3.SCL, IC5.PC1/OC0B/XCK0/SCL, R6.1
- new net SDA_VL53V0X_3V3: IC3.SDA, IC5.PC0/OC0A/SDA, R5.1
- net +3V3: now also C20.1, C21.1, IC3.AVDD, IC3.AVDDVCSEL, R3.2, R4.2, R6.2; no longer C6.1, C7.1, IC2.VCC
- net GND: now also C20.2, C21.2, IC3.AVSSVCSEL, IC3.GND@1, IC3.GND@2, IC3.GND@3, IC3.GND@4; no longer C6.2, C7.2, C8.1, C9.1, IC2.GND, R3.1, R4.1, R6.1, R7.1
- net LED_BLUE_CMD_3V3: now also IC5.TXD0/OC0D/PD3; no longer IC5.PC0/OC0A/SDA
- net LED_GREEN_CMD_3V3: now also IC5.\S\S/PD4; no longer IC5.PC1/OC0B/XCK0/SCL
Other:
- moved on the sheet: R3, R4, R5, R6
